File: analog.kicad_sch (KiCad schematic)
At the start: 36 parts, among them J2 494_OUT, J3 POT, Q2 AO3400A, U1 TL494, U5 LM358

Commit message: +5Vref for softstart, power LED,another connectors
Parts:
- removed J2: 494_OUT, Connector_PinHeader_2.54mm:PinHeader_1x02_P2.54mm_Vertical, symbol Connector_Generic:Conn_01x02
- added C15: 10u, Capacitor_SMD:C_1206_3216Metric_Pad1.33x1.80mm_HandSolder, symbol Device:C
- added J2: ATX, Connector_PinHeader_2.54mm:PinHeader_1x03_P2.54mm_Vertical, symbol Connector_Generic:Conn_01x03
Connections:
- net +5V is gone; now on net +5V_REF: R7.1
- net GND: now also C15.2
- net at C19.1, R13.2, U1.12 (VCC): now also C15.1
- net at U1.11 (C2): now also J2.2 (Pin_2)
- net at U1.8 (C1): now also J2.1 (Pin_1)
- new net +17.5V: J2.3 (Pin_3)
Other:
- note added: "Optional"
- note added: "Optional Filter:f(-3):10 kHz"
- note added: "Remote start: 1 - ON 0 - OFF Rising 10ms"
- note removed: "Filter: f(-3):10 kHz"
- note removed: "Remote start: 1 - ON 0 - OFF Rising 50ms"
- moved on the sheet: C10, C14, C34, C35, C6, C9, J3, R16, R18, R24, R25, R5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
